File: pcb/jumper.kicad_sch (KiCad schematic)
At the start: 0 parts

Commit message: fix: ERC, mark edge connector pins as passive
Parts:
- added H5, H6, H7, H8: MountingHole, MountingHole:MountingHole_3.2mm_M3, symbol Mechanical:MountingHole
