File: pcb/psu.kicad_sch (KiCad schematic)
At the start: 1 part

Commit message: feat: ERC and DRC in CI
Parts:
- J12: renamed from J11; LCSC Part Name S-64L-2.54-5 -> (none); Manufacturer Part S-64L-2.54-5 -> (none); Supplier LCSC -> (none); Supplier Part C9900001011 -> (none)
Changed lines of the file:
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@@
 		(dnp no)
 		(fields_autoplaced yes)
-		(property "Reference" "J11"
+		(property "Reference" "J12"
 			(at 45.72 24.13 0)
 			(effects
@@
 			)
 		)
-		(property "Datasheet" ""
+		(property "Datasheet" "https://github.com/KCORES/KCORES-CSPS-to-ATX-Converter/blob/main/Document/Datasheet/WingTAT%20S-xxM-2.54-x-xx.pdf"
 			(at 45.72 71.12 0)
 			(effects
@@
 		)
 		(property "Description" ""
-			(at 45.72 71.12 0)
-			(effects
-				(font
-					(size 1.27 1.27)
-				)
-				(hide yes)
-			)
-		)
-		(property "Manufacturer Part" "S-64L-2.54-5"
-			(at 45.72 71.12 0)
-			(effects
-				(font
-					(size 1.27 1.27)
-				)
-				(hide yes)
-			)
-		)
-		(property "Supplier Part" "C9900001011"
-			(at 45.72 71.12 0)
-			(effects
-				(font
-					(size 1.27 1.27)
-				)
-				(hide yes)
-			)
-		)
-		(property "Supplier" "LCSC"
-			(at 45.72 71.12 0)
-			(effects
-				(font
-					(size 1.27 1.27)
-				)
-				(hide yes)
-			)
-		)
-		(property "LCSC Part Name" "S-64L-2.54-5"
 			(at 45.72 71.12 0)
 			(effects
@@
 			(project "pdu"
 				(path "/868598ab-f1a7-4d2b-9f5c-b3412115ebb5/83e31ad8-0e16-4075-8c02-9dd13935ed62/576fffd4-855a-483e-987a-07264d2abf3f"
-					(reference "J11")
+					(reference "J12")
 					(unit 1)
 				)
